File: pcb/pinky/nijuni.kicad_sch (KiCad schematic)
At the start: 72 parts, among them J1 MJ-4PP-9, J2 Conn_01x04, J3 Conn_01x02_Female, K1 KEYSW, K10 KEYSW, K11 KEYSW, K12 KEYSW, K13 KEYSW, K14 KEYSW, K15 KEYSW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

Commit message: Added proper footprint dependencies
Parts:
- J1: footprint Keyboard_Components:MJ-4PP-9 -> kbd:MJ-4PP-9
- J2: footprint Keyboard_Components:OLED_DISPLAY_128x32px_0.91in -> kbd:OLED_v2
Changed lines of the file:
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@@
       (effects (font (size 1.27 1.27)) (justify left))
     )
-    (property "Footprint" "Keyboard_Components:OLED_DISPLAY_128x32px_0.91in" (id 2) (at 200.66 71.12 0)
+    (property "Footprint" "kbd:OLED_v2" (id 2) (at 200.66 71.12 0)
       (effects (font (size 1.27 1.27)) hide)
     )
@@
     (property "Reference" "J1" (id 0) (at 149.86 31.115 0))
     (property "Value" "MJ-4PP-9" (id 1) (at 149.86 33.655 0))
-    (property "Footprint" "Keyboard_Components:MJ-4PP-9" (id 2) (at 155.575 34.29 0)
+    (property "Footprint" "kbd:MJ-4PP-9" (id 2) (at 155.575 34.29 0)
       (effects (font (size 1.27 1.27)) hide)
     )
@@
     )
     (path "/f9fbf65c-f051-44ca-8673-b33a76d41a04"
-      (reference "J1") (unit 1) (value "MJ-4PP-9") (footprint "Keyboard_Components:MJ-4PP-9")
+      (reference "J1") (unit 1) (value "MJ-4PP-9") (footprint "kbd:MJ-4PP-9")
     )
     (path "/30e745fe-8230-4e5c-a866-5dee0c1db4aa"
-      (reference "J2") (unit 1) (value "Conn_01x04") (footprint "Keyboard_Components:OLED_DISPLAY_128x32px_0.91in")
+      (reference "J2") (unit 1) (value "Conn_01x04") (footprint "kbd:OLED_v2")
     )
     (path "/c376344d-3f87-44f7-ad86-714ee8048845"
