File: bottom/laser_6col/nijuni-bottom.kicad_pcb (KiCad board)
At the start: 2 copper layers, 134.6 x 95.3 mm, 7 parts

Commit message: Updated laser cutting files
Parts:
- H1, H2, H4, H5, H6, H8, H9: footprint kbd:M2_Hole_TH_mod -> kbd:M2_Hole_Edge_Cut
Changed lines of the file:
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@@
   )
   (net 0 "")
-  (footprint "kbd:M2_Hole_TH_mod" (layer "F.Cu")
+  (footprint "kbd:M2_Hole_Edge_Cut" (layer "F.Cu")
     (at 71.621463 38.074367)
     (property "Sheet file" "rt22-plate.kicad_sch")
     (property "Sheet name" "")
-    (fp_text reference "H4" (at 0 0.5) (layer "F.SilkS")
+    (fp_text reference "H4" (at 0 1.9) (layer "Dwgs.User")
       (effects (font (size 1 1) (thickness 0.15)))
     )
-    (fp_text value "MountingHole" (at 0 -0.5) (layer "F.Fab")
-      (effects (font (size 1 1) (thickness 0.15)))
-    )
-    (fp_text user "${REFERENCE}" (at 0.3 0) (layer "F.Fab")
+    (fp_text value "MountingHole" (at 0 -1.8) (layer "F.Fab")
       (effects (font (size 1 1) (thickness 0.15)))
     )
     (fp_circle (center 0 0) (end 1.15 0) (layer "Edge.Cuts") (width 0.1) (fill none))
-    (pad "" thru_hole circle (at 0 0) (size 4.2 4.2) (drill 2.3) (layers *.Cu *.Mask))
   )
-  (footprint "kbd:M2_Hole_TH_mod" (layer "F.Cu")
+  (footprint "kbd:M2_Hole_Edge_Cut" (layer "F.Cu")
     (at 142.507505 87.19918)
     (property "Sheet file" "rt22-plate.kicad_sch")
     (property "Sheet name" "")
-    (fp_text reference "H9" (at 0 0.5) (layer "F.SilkS")
+    (fp_text reference "H9" (at 0 1.9) (layer "Dwgs.User")
       (effects (font (size 1 1) (thickness 0.15)))
     )
-    (fp_text value "MountingHole" (at 0 -0.5) (layer "F.Fab")
-      (effects (font (size 1 1) (thickness 0.15)))
-    )
-    (fp_text user "${REFERENCE}" (at 0.3 0) (layer "F.Fab")
+    (fp_text value "MountingHole" (at 0 -1.8) (layer "F.Fab")
       (effects (font (size 1 1) (thickness 0.15)))
     )
     (fp_circle (center 0 0) (end 1.15 0) (layer "Edge.Cuts") (width 0.1) (fill none))
-    (pad "" thru_hole circle (at 0 0) (size 4.2 4.2) (drill 2.3) (layers *.Cu *.Mask))
   )
-  (footprint "kbd:M2_Hole_TH_mod" (layer "F.Cu")
+  (footprint "kbd:M2_Hole_Edge_Cut" (layer "F.Cu")
     (at 51.821463 66.574367)
     (property "Sheet file" "rt22-plate.kicad_sch")
     (property "Sheet name" "")
-    (fp_text reference "H2" (at 0 0.5) (layer "F.SilkS")
+    (fp_text reference "H2" (at 0 1.9) (layer "Dwgs.User")
       (effects (font (size 1 1) (thickness 0.15)))
     )
-    (fp_text value "MountingHole" (at 0 -0.5) (layer "F.Fab")
-      (effects (font (size 1 1) (thickness 0.15)))
-    )
-    (fp_text user "${REFERENCE}" (at 0.3 0) (layer "F.Fab")
+    (fp_text value "MountingHole" (at 0 -1.8) (layer "F.Fab")
       (effects (font (size 1 1) (thickness 0.15)))
     )
     (fp_circle (center 0 0) (end 1.15 0) (layer "Edge.Cuts") (width 0.1) (fill none))
-    (pad "" thru_hole circle (at 0 0) (size 4.2 4.2) (drill 2.3) (layers *.Cu *.Mask))
   )
-  (footprint "kbd:M2_Hole_TH_mod" (layer "F.Cu")
+  (footprint "kbd:M2_Hole_Edge_Cut" (layer "F.Cu")
     (at 128.721463 40.374367)
     (property "Sheet file" "rt22-plate.kicad_sch")
     (property "Sheet name" "")
-    (fp_text reference "H8" (at 0 0.5) (layer "F.SilkS")
+    (fp_text reference "H8" (at 0 1.9) (layer "Dwgs.User")
       (effects (font (size 1 1) (thickness 0.15)))
     )
-    (fp_text value "MountingHole" (at 0 -0.5) (layer "F.Fab")
-      (effects (font (size 1 1) (thickness 0.15)))
-    )
-    (fp_text user "${REFERENCE}" (at 0.3 0) (layer "F.Fab")
+    (fp_text value "MountingHole" (at 0 -1.8) (layer "F.Fab")
       (effects (font (size 1 1) (thickness 0.15)))
     )
     (fp_circle (center 0 0) (end 1.15 0) (layer "Edge.Cuts") (width 0.1) (fill none))
-    (pad "" thru_hole circle (at 0 0) (size 4.2 4.2) (drill 2.3) (layers *.Cu *.Mask))
   )
-  (footprint "kbd:M2_Hole_TH_mod" (layer "F.Cu")
+  (footprint "kbd:M2_Hole_Edge_Cut" (layer "F.Cu")
     (at 97.421463 75.774367)
     (property "Sheet file" "rt22-plate.kicad_sch")
     (property "Sheet name" "")
-    (fp_text reference "H6" (at 0 0.5) (layer "F.SilkS")
+    (fp_text reference "H6" (at 0 1.9) (layer "Dwgs.User")
       (effects (font (size 1 1) (thickness 0.15)))
     )
-    (fp_text value "MountingHole" (at 0 -0.5) (layer "F.Fab")
-      (effects (font (size 1 1) (thickness 0.15)))
-    )
-    (fp_text user "${REFERENCE}" (at 0.3 0) (layer "F.Fab")
+    (fp_text value "MountingHole" (at 0 -1.8) (layer "F.Fab")
       (effects (font (size 1 1) (thickness 0.15)))
     )
     (fp_circle (center 0 0) (end 1.15 0) (layer "Edge.Cuts") (width 0.1) (fill none))
-    (pad "" thru_hole circle (at 0 0) (size 4.2 4.2) (drill 2.3) (layers *.Cu *.Mask))
   )
-  (footprint "kbd:M2_Hole_TH_mod" (layer "F.Cu")
+  (footprint "kbd:M2_Hole_Edge_Cut" (layer "F.Cu")
     (at 51.721463 47.574367)
     (property "Sheet file" "rt22-plate.kicad_sch")
     (property "Sheet name" "")
-    (fp_text reference "H1" (at 0 0.5) (layer "F.SilkS")
+    (fp_text reference "H1" (at 0 1.9) (layer "Dwgs.User")
       (effects (font (size 1 1) (thickness 0.15)))
     )
-    (fp_text value "MountingHole" (at 0 -0.5) (layer "F.Fab")
-      (effects (font (size 1 1) (thickness 0.15)))
-    )
-    (fp_text user "${REFERENCE}" (at 0.3 0) (layer "F.Fab")
+    (fp_text value "MountingHole" (at 0 -1.8) (layer "F.Fab")
       (effects (font (size 1 1) (thickness 0.15)))
     )
     (fp_circle (center 0 0) (end 1.15 0) (layer "Edge.Cuts") (width 0.1) (fill none))
-    (pad "" thru_hole circle (at 0 0) (size 4.2 4.2) (drill 2.3) (layers *.Cu *.Mask))
   )
-  (footprint "kbd:M2_Hole_TH_mod" (layer "F.Cu")
+  (footprint "kbd:M2_Hole_Edge_Cut" (layer "F.Cu")
     (at 71.721463 79.774367)
     (property "Sheet file" "rt22-plate.kicad_sch")
     (property "Sheet name" "")
-    (fp_text reference "H5" (at 0 0.5) (layer "F.SilkS")
+    (fp_text reference "H5" (at 0 1.9) (layer "Dwgs.User")
       (effects (font (size 1 1) (thickness 0.15)))
     )
-    (fp_text value "MountingHole" (at 0 -0.5) (layer "F.Fab")
-      (effects (font (size 1 1) (thickness 0.15)))
-    )
-    (fp_text user "${REFERENCE}" (at 0.3 0) (layer "F.Fab")
+    (fp_text value "MountingHole" (at 0 -1.8) (layer "F.Fab")
       (effects (font (size 1 1) (thickness 0.15)))
     )
     (fp_circle (center 0 0) (end 1.15 0) (layer "Edge.Cuts") (width 0.1) (fill none))
-    (pad "" thru_hole circle (at 0 0) (size 4.2 4.2) (drill 2.3) (layers *.Cu *.Mask))
   )
   (gr_circle (center 109.221463 86.099097) (end 108.721463 86.099097) (layer "Cmts.User") (width 0.2) (fill none))
