File: bottom/laser_pinky/nijuni-bottom.kicad_pcb (KiCad board)
At the start: 2 copper layers, 153.6 x 95.3 mm, 8 parts

Commit message: Updated laser cutting files
Parts:
- H1, H2, H3, H4, H5, H6, H8, H9: footprint kbd:M2_Hole_TH_mod -> kbd:M2_Hole_Edge_Cut
